Commit message: steering on wheels

File: car_gazebo_models/models/platforms/car/body/wheel.xacro (robot description, xacro)
@@ -12,8 +12,10 @@
     <xacro:property name="cap_length" value="0.005" />
     <!-- Mount -->
-    <joint name="wheel_mount_${side}_joint" type="fixed">
+    <joint name="wheel_mount_${side}_joint" type="revolute">
         <origin xyz="${xyz}" rpy="${rpy}"/>
         <parent link="${parent}"/>
         <child link="wheel_mount_${side}"/>
+        <axis xyz="0 1 0"/>
+        <limit effort="50" velocity="50" lower= "${-M_PI}" upper="${M_PI}" /> <!--velocity="5" -->
     </joint>
     <link name="wheel_mount_${side}">

Commit message: moves

File: car_gazebo_models/models/platforms/car/body/wheel.xacro (robot description, xacro)
@@ -12,10 +12,10 @@
     <xacro:property name="cap_length" value="0.005" />
     <!-- Mount -->
-    <joint name="wheel_mount_${side}_joint" type="revolute">
+    <joint name="wheel_mount_${side}_joint" type="fixed">  <!--fixed/revolute -->
         <origin xyz="${xyz}" rpy="${rpy}"/>
         <parent link="${parent}"/>
         <child link="wheel_mount_${side}"/>
         <axis xyz="0 1 0"/>
-        <limit effort="50" velocity="50" lower= "${-M_PI}" upper="${M_PI}" /> <!--velocity="5" -->
+        <limit effort="50" velocity="50" lower= "${-M_PI}" upper="${M_PI}" />
     </joint>
     <link name="wheel_mount_${side}">
@@ -61,5 +61,5 @@
         <child link="wheel_axis_${side}"/>
         <axis xyz="0 0 1"/>
-          <dynamics damping="0.0001" friction="0.0"/>
+          <dynamics damping="0.000" friction="0.0"/>
     </joint>
     <link name="wheel_axis_${side}">

Commit message: Refactor xacor

File: car_gazebo_models/models/platforms/car/body/wheel.xacro (robot description, xacro)
@@ -56,7 +56,5 @@
     </link>
     <!-- axis -->
-    <joint name="wheel_axis_${side}_joint" type="continuous">/3
-        ******************------------------+
-        -
+    <joint name="wheel_axis_${side}_joint" type="continuous">
         <origin xyz=" 0 0 ${steering_radius}" rpy="0 0 0"/>
         <parent link="wheel_steering_${side}"/>
@@ -90,5 +88,5 @@
     <link name="wheel_${side}">
         <visual>
-            <origin xyz="0 0 ${wheel_length/2}" rpy="0 0 0"/>
+            <origin xyz="0 0 ${wheel_length/2}" rpy="${M_PI/2} 0 0"/>
             <geometry>
                 <cylinder radius="${wheel_radius}" length="${wheel_length}"/>

Commit message: undo change

File: car_gazebo_models/models/platforms/car/body/wheel.xacro (robot description, xacro)
@@ -88,5 +88,5 @@
     <link name="wheel_${side}">
         <visual>
-            <origin xyz="0 0 ${wheel_length/2}" rpy="${M_PI/2} 0 0"/>
+            <origin xyz="0 0 ${wheel_length/2}" rpy="0 0 0"/>
             <geometry>
                 <cylinder radius="${wheel_radius}" length="${wheel_length}"/>
