Commit message: car without steering working

File: car_gazebo_models/models/platforms/car/body/body.xacro (robot description, xacro)
@@ -3,5 +3,6 @@
   <xacro:include filename="inertia_tensors.xacro"/>
   <xacro:include filename="chassis.xacro"/>
-  <xacro:property name="wheel_radius" value="0.097" />
+  <xacro:include filename="wheel.xacro"/>
+  <xacro:property name="wheel_radius" value="0.0325" />
   <xacro:property name="M_PI" value="3.1415926535897931" />
   <xacro:macro name="car_body" params="name parent">
@@ -10,4 +11,8 @@
     <!-- Chassis -->
     <xacro:car_chassis name="${name}" parent="${parent}" xyz="0 0 0.068" rpy="0 0 0"/>
+    <xacro:wheel side="rear_left"  parent="${parent}"   xyz="0    -0.055 ${wheel_radius}" rpy="+${pi/2} 0 0" radius="${wheel_radius}"/>
+    <xacro:wheel side="rear_right" parent="${parent}"   xyz="0    +0.055 ${wheel_radius}" rpy="-${pi/2} 0 0" radius="${wheel_radius}"/>
+    <xacro:wheel side="front_left"  parent="${parent}"  xyz="0.26 -0.055 ${wheel_radius}" rpy="+${pi/2} 0 0" radius="${wheel_radius}"/>
+    <xacro:wheel side="front_right" parent="${parent}"  xyz="0.26 +0.055 ${wheel_radius}" rpy="-${pi/2} 0 0" radius="${wheel_radius}"/>
   </xacro:macro>
 </robot>

File: car_gazebo_models/models/platforms/car/body/chassis.xacro (robot description, xacro)
@@ -1,6 +1,4 @@
 <?xml version="1.0"?>
 <robot xmlns:xacro="http://ros.org/wiki/xacro">
-  <xacro:property name="bottom_plate_box_size"    value=" 0.26  0.08  0.02" />
-  <xacro:property name="bottom_plate_origin"      value="-0.13  0.00 -0.02" />
   <xacro:macro name="inertia_box" params="x y z mass">
       <mass value="${mass}" />
@@ -9,5 +7,8 @@
         izz="${0.0833333 * mass * (x*x + y*y)}" />
   </xacro:macro>
-  <xacro:macro name="car_chassis" params="name parent xyz rpy model_dir:=^">
+  <xacro:macro name="car_chassis" params="name parent xyz rpy">
+  <xacro:property name="plate_x"    value="0.26" />
+  <xacro:property name="plate_y"    value="0.08" />
+  <xacro:property name="plate_z"    value="0.02" />
     <!-- Chassis -->
     <joint name="${parent}_${name}_joint" type="fixed">
@@ -18,21 +19,21 @@
     <link name="${name}">
         <visual>
-        <origin xyz="${bottom_plate_origin}" rpy="0 0 0"/>
-        <geometry>
-            <box size="${bottom_plate_box_size}"/>
-        </geometry>
-        <material name="ChassisRed">
-            <color rgba="0.851 0.0 0.0 1.0"/>
-        </material>
+            <origin xyz="${plate_x/2} 0 -${plate_z}" rpy="0 0 0"/>
+            <geometry>
+                <box size="${plate_x} ${plate_y} ${plate_z}"/>
+            </geometry>
+            <material name="ChassisRed">
+                <color rgba="0.851 0.0 0.0 1.0"/>
+            </material>
         </visual>
         <collision>
-            <origin xyz="${bottom_plate_origin}" rpy="0 0 0"/>
+            <origin xyz="${plate_x/2} 0 -${plate_z}" rpy="0 0 0"/>
             <geometry>
-                <box size="${bottom_plate_box_size}"/>
+                <box size="${plate_x} ${plate_y} ${plate_z}"/>
             </geometry>
         </collision>
         <inertial>
-            <origin xyz="${bottom_plate_origin}" />
-            <xacro:inertia_box x="0.26" y="0.08"  z="0.02" mass="0.01" />
+            <origin xyz="${plate_x/2} 0 -${plate_z}" />
+            <xacro:inertia_box x="${plate_x}" y="${plate_y}"  z="${plate_z}" mass="0.01" />
         </inertial>
     </link>

File: car_gazebo_models/models/platforms/car/body/wheel.xacro (robot description, xacro)
@@ -1,19 +1,18 @@
 <?xml version="1.0"?>
 <robot xmlns:xacro="http://ros.org/wiki/xacro">
-  <xacro:macro name="inertia_box" params="x y z mass">
-      <mass value="${mass}" />
-      <inertia ixx="${0.0833333 * mass * (y*y + z*z)}" ixy="0.0" ixz="0.0"
-        iyy="${0.0833333 * mass * (x*x + z*z)}" iyz="0.0"
-        izz="${0.0833333 * mass * (x*x + y*y)}" />
-  </xacro:macro>
-  <xacro:macro name="car_wheel" params="side parent xyz rpy radius model_dir:=^ **contact_data">
-    <!-- Hubcap Mount -->
-    <joint name="${side}_hub_mount_joint" type="fixed">
+  <xacro:macro name="wheel" params="side parent xyz rpy radius">
+    <xacro:property name="mount_lenth" value="0.01" />
+    <xacro:property name="mount_radius" value="0.02" />
+    <xacro:property name="axis_lenth" value="0.01" />
+    <xacro:property name="axis_radius" value="0.01" />
+    <xacro:property name="wheel_lenth" value="0.025" />
+    <xacro:property name="wheel_radius" value="${radius}" />
+    <!-- Mount -->
+    <joint name="wheel_mount_${side}_joint" type="fixed">
         <origin xyz="${xyz}" rpy="${rpy}"/>
         <parent link="${parent}"/>
-        <child link="${side}_hub_mount"/>
-        <axis xyz="0 1 0"/>
+        <child link="wheel_mount_${side}"/>
     </joint>
-    <link name="${side}_hub_mount">
+    <link name="wheel_mount_${side}">
         <inertial>
             <mass value="0.01"/>
@@ -22,13 +21,63 @@
         </inertial>
         <visual>
-            <origin xyz="0 0 0" rpy="0 0 0"/>
+            <origin xyz="0 0 ${mount_lenth/2}" rpy="0 0 0"/>
             <geometry>
-                <box size="0.001 0.001 0.001"/>
+                <cylinder radius="${mount_radius}" length="${mount_lenth}"/>
             </geometry>
         </visual>
         <collision>
-            <origin xyz="0 0 0" rpy="0 0 0"/>
+            <origin xyz="0 0 ${mount_lenth/2} " rpy="0 0 0"/>
             <geometry>
-                <box size="0.001 0.001 0.001"/>
+                <cylinder radius="${mount_radius}" length="${mount_lenth}"/>
+            </geometry>
+        </collision>
+    </link>
+    <!-- axis -->
+    <joint name="wheel_axis_${side}_joint" type="fixed">
+        <origin xyz=" 0 0 ${mount_lenth}" rpy="0 0 0"/>
+        <parent link="wheel_mount_${side}"/>
+        <child link="wheel_axis_${side}"/>
+    </joint>
+    <link name="wheel_axis_${side}">
+        <inertial>
+            <mass value="0.01"/>
+            <origin xyz="0 0 0"/>
+            <inertia ixx="0.012411765597" ixy="0" ixz="0" iyy="0.015218160428" iyz="0" izz="0.011763977943"/>
+        </inertial>
+        <visual>
+            <origin xyz="0 0 ${axis_lenth/2}" rpy="0 0 0"/>
+            <geometry>
+                <cylinder radius="${axis_radius}" length="${axis_lenth}"/>
+            </geometry>
+        </visual>
+        <collision>
+            <origin xyz="0 0 ${axis_lenth/2}" rpy="0 0 0"/>
+            <geometry>
+                <cylinder radius="${axis_radius}" length="${axis_lenth}"/>
+            </geometry>
+        </collision>
+    </link>
+    <!-- Wheel -->
+    <joint name="wheel_${side}_joint" type="fixed">
+        <origin xyz=" 0 0 ${axis_lenth}" rpy="0 0 0"/>
+        <parent link="wheel_axis_${side}"/>
+        <child link="wheel_${side}"/>
+    </joint>
+    <link name="wheel_${side}">
+        <inertial>
+            <mass value="0.01"/>
+            <origin xyz="0 0 0"/>
+            <inertia ixx="0.012411765597" ixy="0" ixz="0" iyy="0.015218160428" iyz="0" izz="0.011763977943"/>
+        </inertial>
+        <visual>
+            <origin xyz="0 0 ${wheel_lenth/2}" rpy="0 0 0"/>
+            <geometry>
+                <cylinder radius="${wheel_radius}" length="${wheel_lenth}"/>
+            </geometry>
+        </visual>
+        <collision>
+            <origin xyz="0 0 ${wheel_lenth/2}" rpy="0 0 0"/>
+            <geometry>
+                <cylinder radius="${wheel_radius}" length="${wheel_lenth}"/>
             </geometry>
         </collision>

Commit message: plugin added

File: car_gazebo_models/models/platforms/car/body/body.xacro (robot description, xacro)
@@ -6,4 +6,10 @@
   <xacro:property name="wheel_radius" value="0.0325" />
   <xacro:property name="M_PI" value="3.1415926535897931" />
+  <xacro:macro name="wheels_steering">
+    <gazebo>
+        <plugin name="wheels_steering_controller" filename="libgazebo_ros_wheels_steerable.so">
+        </plugin>
+    </gazebo>
+  </xacro:macro>
   <xacro:macro name="car_body" params="name parent">
     <!-- base_link -->
@@ -11,8 +17,10 @@
     <!-- Chassis -->
     <xacro:car_chassis name="${name}" parent="${parent}" xyz="0 0 0.068" rpy="0 0 0"/>
-    <xacro:wheel side="rear_left"  parent="${parent}"   xyz="0    -0.055 ${wheel_radius}" rpy="+${pi/2} 0 0" radius="${wheel_radius}"/>
-    <xacro:wheel side="rear_right" parent="${parent}"   xyz="0    +0.055 ${wheel_radius}" rpy="-${pi/2} 0 0" radius="${wheel_radius}"/>
-    <xacro:wheel side="front_left"  parent="${parent}"  xyz="0.26 -0.055 ${wheel_radius}" rpy="+${pi/2} 0 0" radius="${wheel_radius}"/>
-    <xacro:wheel side="front_right" parent="${parent}"  xyz="0.26 +0.055 ${wheel_radius}" rpy="-${pi/2} 0 0" radius="${wheel_radius}"/>
+    <xacro:wheel side="rear_left"   parent="${parent}"   xyz="0    -0.055 ${wheel_radius}" rpy="+${pi/2} 0 0" radius="${wheel_radius}"/>
+    <xacro:wheel side="rear_right"  parent="${parent}"   xyz="0    +0.055 ${wheel_radius}" rpy="-${pi/2} 0 0" radius="${wheel_radius}"/>
+    <xacro:wheel side="front_left"  parent="${parent}"   xyz="0.26 -0.055 ${wheel_radius}" rpy="+${pi/2} 0 0" radius="${wheel_radius}"/>
+    <xacro:wheel side="front_right" parent="${parent}"   xyz="0.26 +0.055 ${wheel_radius}" rpy="-${pi/2} 0 0" radius="${wheel_radius}"/>
+    <!-- Motor plugin -->
+    <xacro:wheels_steering />
   </xacro:macro>
 </robot>

Commit message: driving and steering working

File: car_gazebo_models/models/platforms/car/body/body.xacro (robot description, xacro)
@@ -6,10 +6,4 @@
   <xacro:property name="wheel_radius" value="0.0325" />
   <xacro:property name="M_PI" value="3.1415926535897931" />
-  <xacro:macro name="wheels_steering">
-    <gazebo>
-        <plugin name="wheels_steering_controller" filename="libgazebo_ros_wheels_steerable.so">
-        </plugin>
-    </gazebo>
-  </xacro:macro>
   <xacro:macro name="car_body" params="name parent">
     <!-- base_link -->
@@ -17,8 +11,8 @@
     <!-- Chassis -->
     <xacro:car_chassis name="${name}" parent="${parent}" xyz="0 0 0.068" rpy="0 0 0"/>
-    <xacro:wheel side="rear_left"   parent="${parent}"   xyz="0    -0.055 ${wheel_radius}" rpy="+${pi/2} 0 0" radius="${wheel_radius}"/>
-    <xacro:wheel side="rear_right"  parent="${parent}"   xyz="0    +0.055 ${wheel_radius}" rpy="-${pi/2} 0 0" radius="${wheel_radius}"/>
-    <xacro:wheel side="front_left"  parent="${parent}"   xyz="0.26 -0.055 ${wheel_radius}" rpy="+${pi/2} 0 0" radius="${wheel_radius}"/>
-    <xacro:wheel side="front_right" parent="${parent}"   xyz="0.26 +0.055 ${wheel_radius}" rpy="-${pi/2} 0 0" radius="${wheel_radius}"/>
+    <xacro:wheel side="rear_left"   parent="${parent}"   xyz="0    -0.055 ${wheel_radius}" rpy="+${pi/2} 0 0" radius="${wheel_radius}"  steering="fixed"/>
+    <xacro:wheel side="rear_right"  parent="${parent}"   xyz="0    +0.055 ${wheel_radius}" rpy="-${pi/2} 0 0" radius="${wheel_radius}"  steering="fixed"/>
+    <xacro:wheel side="front_left"  parent="${parent}"   xyz="0.26 -0.055 ${wheel_radius}" rpy="+${pi/2} 0 0" radius="${wheel_radius}"  steering="revolute"/>
+    <xacro:wheel side="front_right" parent="${parent}"   xyz="0.26 +0.055 ${wheel_radius}" rpy="-${pi/2} 0 0" radius="${wheel_radius}"  steering="revolute"/>
     <!-- Motor plugin -->
     <xacro:wheels_steering />

File: car_gazebo_models/models/platforms/car/body/wheel.xacro (robot description, xacro)
@@ -1,5 +1,5 @@
 <?xml version="1.0"?>
 <robot xmlns:xacro="http://ros.org/wiki/xacro">
-  <xacro:macro name="wheel" params="side parent xyz rpy radius">
+  <xacro:macro name="wheel" params="side parent xyz rpy radius steering">
     <xacro:property name="mount_size" value="0.01" />
     <xacro:property name="steering_length" value="0.03" />
@@ -12,5 +12,5 @@
     <xacro:property name="cap_length" value="0.005" />
     <!-- Mount -->
-    <joint name="wheel_mount_${side}_joint" type="fixed">  <!--fixed/revolute -->
+    <joint name="wheel_mount_${side}_joint" type="${steering}">  <!--fixed/revolute -->
         <origin xyz="${xyz}" rpy="${rpy}"/>
         <parent link="${parent}"/>
@@ -56,5 +56,7 @@
     </link>
     <!-- axis -->
-    <joint name="wheel_axis_${side}_joint" type="continuous">
+    <joint name="wheel_axis_${side}_joint" type="continuous">/3
+        ******************------------------+
+        -
         <origin xyz=" 0 0 ${steering_radius}" rpy="0 0 0"/>
         <parent link="wheel_steering_${side}"/>

File: car_gazebo_models/models/platforms/car/main.xacro (robot description, xacro)
@@ -6,4 +6,5 @@
   <!-- Import Rviz colors -->
   <xacro:include filename="$(arg model_dir)/materials.xacro" />
+  <xacro:include filename="$(arg model_dir)/$(arg platform_dir)/plugins.xacro" />
   <!-- Import platform -->
   <xacro:property name="model_dir" value="$(arg model_dir)/$(arg platform_dir)/body"/>

File: car_gazebo_models/models/platforms/car/plugins.xacro (robot description, xacro)
@@ -1,57 +1,20 @@
 <?xml version="1.0"?>
 <robot xmlns:xacro="http://ros.org/wiki/xacro">
-  <xacro:macro name="diff_joints_state_publisher" params="ns">
+  <xacro:macro name="wheels_steering">
     <gazebo>
-        <plugin name="joint_state_publisher" filename="libgazebo_ros_joint_state_publisher.so">
-          <robotNamespace>${ns}</robotNamespace>
-          <jointName>chassis_swivel_joint, swivel_wheel_joint, left_hub_joint, right_hub_joint</jointName>
-          <updateRate>20.0</updateRate>
-          <alwaysOn>true</alwaysOn>
+        <plugin name="wheels_steering_controller" filename="libgazebo_ros_wheels_steerable.so">
+            <rosDebugLevel>Debug</rosDebugLevel>
+            <rosDebugLevel>Debug</rosDebugLevel>
+            <topicOdom>odom</topicOdom>
+            <frameBase>odom</frameBase>
+            <frameOdom>odom</frameOdom>
+            <topicTwist>cmd_vel</topicTwist>
+            <jointRearLeft>wheel_axis_rear_left_joint</jointRearLeft>
+            <jointRearRight>wheel_axis_rear_right_joint</jointRearRight>
+            <jointSteeringLeft>wheel_mount_front_left_joint</jointSteeringLeft>
+            <jointSteeringRight>wheel_mount_front_right_joint</jointSteeringRight>
+            <torqueMaxWheel>5</torqueMaxWheel>
         </plugin>
     </gazebo>
   </xacro:macro>
-  <xacro:macro name="differential_drive">
-    <gazebo>
-        <plugin name="differential_drive_controller" filename="libtuw_gazebo_ros_diff_drive.so">
-	      <robotNamespace></robotNamespace>
-          <rosDebugLevel>Debug</rosDebugLevel>
-          <alwaysOn>true</alwaysOn>
-          <alwaysOn>true</alwaysOn>
-	      <updateRate>20.0</updateRate>
-	      <robotBaseFrame>base_link</robotBaseFrame>
-	      <odometryFrame>odom</odometryFrame>
-	      <commandTopic>cmd_vel</commandTopic>
-          <odometryTopic>odom</odometryTopic>
-          <!-- odom source world or encoder, world uses the simulated ground truth and encoder the wheel odometry -->
-          <odometrySource>encoder</odometrySource>
-          <leftJoint>left_hub_joint</leftJoint>
-          <rightJoint>right_hub_joint</rightJoint>
-          <wheelSeparation>0.3</wheelSeparation>
-          <wheelDiameter>0.18</wheelDiameter>
-          <wheelTorque>10</wheelTorque>
-          <wheelAcceleration>1.5</wheelAcceleration>
-          <publishTf>true</publishTf>
-	      <publishWheelTF>true</publishWheelTF>
-          <publishWheelJointState>true</publishWheelJointState>
-        </plugin>
-    </gazebo>
-  </xacro:macro>
-  <xacro:macro name="iws_joints_state_publisher" params="ns">
-	<gazebo>
-	  <plugin name="joint_state_publisher" filename="libgazebo_ros_joint_state_publisher.so">
-		<robotNamespace>${ns}</robotNamespace>
-		<jointName>chassis_swivel_joint, swivel_wheel_joint</jointName>
-		<updateRate>50.0</updateRate>
-		<alwaysOn>true</alwaysOn>
-	  </plugin>
-	</gazebo>
-  </xacro:macro>
-  <xacro:include filename="plugins_param.xacro"/>
-  <xacro:macro name="iws_drive">
-	<gazebo>
-	  <plugin name="tuw_gazebo_ros_bridge_model_plugin" filename="libtuw_gazebo_ros_bridge_model.so">
-        <xacro:insert_block name="IWSPluginsData" />
-	  </plugin>
-	</gazebo>
-  </xacro:macro>
 </robot>

Commit message: Use full model for view

File: car_gazebo_models/models/platforms/car/body/body.xacro (robot description, xacro)
@@ -3,5 +3,4 @@
   <xacro:include filename="inertia_tensors.xacro"/>
   <xacro:include filename="chassis.xacro"/>
-  <xacro:include filename="top.xacro"/>
   <xacro:include filename="wheel.xacro"/>
   <xacro:property name="wheel_radius" value="0.0325" />
@@ -11,7 +10,5 @@
     <link name="${parent}"/>
     <!-- Chassis -->
-    <xacro:car_chassis name="${name}" parent="${parent}" xyz="0 0 0.068" rpy="0 0 0"/>
-    <!-- Top -->
-    <xacro:car_top name="top_chassis" parent="${parent}" xyz="0 0 0.068" rpy="0 0 0"/>
+    <xacro:car_chassis name="${name}" parent="${parent}" xyz="0.13 0 0.068" rpy="0 0 ${M_PI}"/>
     <!-- Wheel -->
     <xacro:wheel side="rear_left"   parent="${parent}"   xyz="0    -0.055 ${wheel_radius}" rpy="+${pi/2} 0 0" radius="${wheel_radius}"  steering="fixed"/>

File: car_gazebo_models/models/platforms/car/body/chassis.xacro (robot description, xacro)
@@ -15,5 +15,5 @@
             <origin xyz="${plate_x/2} 0 -${plate_z}" rpy="0 0 0"/>
             <geometry>
-                <mesh scale="1 1 1" filename="file://$(arg model_dir)$(arg platform_dir)/body/meshes/car/Bodenplatte.dae"/>
+                <mesh scale="1 1 1" filename="file://$(arg model_dir)$(arg platform_dir)/body/meshes/car.dae/car.dae"/>
                 <!--<box size="${plate_x} ${plate_y} ${plate_z}"/>-->
             </geometry>

Commit message: add odom

File: car_gazebo_models/models/platforms/car/body/body.xacro (robot description, xacro)
@@ -17,5 +17,5 @@
     <xacro:wheel side="front_right" parent="${parent}"   xyz="0.26 +0.055 ${wheel_radius}" rpy="-${pi/2} 0 0" radius="${wheel_radius}"  steering="revolute"/>
     <!-- Motor plugin -->
-    <xacro:wheels_steering />
+    <xacro:wheels_steering radius="${wheel_radius}"/>
   </xacro:macro>
 </robot>

File: car_gazebo_models/models/platforms/car/plugins.xacro (robot description, xacro)
@@ -1,5 +1,6 @@
 <?xml version="1.0"?>
 <robot xmlns:xacro="http://ros.org/wiki/xacro">
-  <xacro:macro name="wheels_steering">
+  <xacro:macro name="wheels_steering" params="radius">
+  <xacro:property name="wheel_radius" value="${radius}" />
     <gazebo>
         <plugin name="wheels_steering_controller" filename="libgazebo_ros_wheels_steerable.so">
@@ -25,4 +26,5 @@
             <pidI>10.0</pidI>
             <pidD>1.0</pidD>
+            <wheelRadius>${wheel_radius}</wheelRadius>
         </plugin>
     </gazebo>

Commit message: Adapt weights and publish angles

File: car_gazebo_models/models/platforms/car/body/body.xacro (robot description, xacro)
@@ -4,5 +4,5 @@
   <xacro:include filename="chassis.xacro"/>
   <xacro:include filename="wheel.xacro"/>
-  <xacro:property name="wheel_radius" value="0.0325" />
+  <xacro:property name="wheel_radius" value="0.03225" />
   <xacro:property name="M_PI" value="3.1415926535897931" />
   <xacro:macro name="car_body" params="name parent">

File: car_gazebo_models/models/platforms/car/body/chassis.xacro (robot description, xacro)
@@ -23,11 +23,11 @@
         </visual>
         <collision>
-            <origin xyz="${plate_x/2} 0 -${plate_z}" rpy="0 0 0"/>
+            <origin xyz="0 0 -${plate_z}" rpy="0 0 0"/>
             <geometry>
                 <box size="${plate_x} ${plate_y} ${plate_z}"/>
             </geometry>
         </collision>
-        <xacro:box_inertial_with_origin x="${plate_x}" y="${plate_y}"  z="${plate_z}" mass="0.01">
-            <origin xyz="${plate_x/2} 0 -${plate_z}" />
+        <xacro:box_inertial_with_origin x="${plate_x}" y="${plate_y}"  z="${plate_z}" mass="0.970">
+            <origin xyz="0 0 -${plate_z}" />
         </xacro:box_inertial_with_origin>
     </link>

File: car_gazebo_models/models/platforms/car/body/wheel.xacro (robot description, xacro)
@@ -7,5 +7,5 @@
     <xacro:property name="axis_length" value="0.01" />
     <xacro:property name="axis_radius" value="0.01" />
-    <xacro:property name="wheel_length" value="0.025" />
+    <xacro:property name="wheel_length" value="0.026" />
     <xacro:property name="wheel_radius" value="${radius}" />
     <xacro:property name="cap_size" value="0.01" />
@@ -35,5 +35,5 @@
     <link name="wheel_steering_${side}">
         <inertial>
-            <mass value="0.01"/>
+            <mass value="0.001"/>
             <origin xyz="0 0 0"/>
             <inertia ixx="0.012411765597" ixy="0" ixz="0" iyy="0.015218160428" iyz="0" izz="0.011763977943"/>
@@ -51,5 +51,5 @@
             </geometry>
         </collision>
-        <xacro:cylinder_inertial_with_origin radius="${axis_radius}" length="${steering_length}"  mass="0.01">
+        <xacro:cylinder_inertial_with_origin radius="${axis_radius}" length="${steering_length}"  mass="0.001">
             <origin xyz="0 0 ${steering_radius/2}" rpy="0 0 0"/>
         </xacro:cylinder_inertial_with_origin>
@@ -76,5 +76,5 @@
             </geometry>
         </collision>
-        <xacro:cylinder_inertial_with_origin radius="${axis_radius}" length="${axis_length}"  mass="0.01">
+        <xacro:cylinder_inertial_with_origin radius="${axis_radius}" length="${axis_length}"  mass="0.1135">
             <origin xyz="0 0 ${axis_length/2}" rpy="0 0 0"/>
         </xacro:cylinder_inertial_with_origin>
@@ -99,5 +99,5 @@
             </geometry>
         </collision>
-        <xacro:cylinder_inertial_with_origin radius="${wheel_radius}" length="${wheel_length}"  mass="0.1">
+        <xacro:cylinder_inertial_with_origin radius="${wheel_radius}" length="${wheel_length}"  mass="0.026">
             <origin xyz="0 0 ${wheel_length/2}" rpy="0 0 0"/>
         </xacro:cylinder_inertial_with_origin>

File: car_gazebo_models/models/platforms/car/plugins.xacro (robot description, xacro)
@@ -24,8 +24,8 @@
             <maxSteeringAngle>0.5235987756</maxSteeringAngle>
             <!--PID controller parameter-->
-            <maxEffortSteeringPid>100.0</maxEffortSteeringPid>
-            <pidP>100.0</pidP>
-            <pidI>10.0</pidI>
-            <pidD>1.0</pidD>
+            <maxEffortSteeringPid>1000.0</maxEffortSteeringPid>
+            <pidP>5.0</pidP>
+            <pidI>0.0</pidI>
+            <pidD>0.0</pidD>
             <wheelRadius>${wheel_radius}</wheelRadius>
         </plugin>
