Commit message: Abgabe Sommersemester 2021

File: car_gazebo_models/models/platforms/car/body/body.xacro (robot description, xacro)
@@ -6,17 +6,30 @@
   <xacro:property name="wheel_radius" value="0.03225" />
   <xacro:property name="M_PI" value="3.1415926535897931" />
-  <xacro:macro name="car_body" params="name namespace parent">
+  <xacro:include filename="$(find realsense2_description)/urdf/_d435.urdf.xacro" />
+  <xacro:arg name="name" default="camera" />
+  <xacro:arg name="topics_ns" default="camera" />
+  <xacro:arg name="use_nominal_extrinsics" default="true" />
+  <xacro:arg name="publish_pointcloud" default="true" />
+  <xacro:arg name="add_plug" default="false" />
+  <xacro:macro name="car_body" params="name parent">
     <!-- base_link -->
-    <link name="${namespace}/${parent}"/>
+    <link name="${parent}"/>
     <!-- Chassis -->
-    <xacro:car_chassis name="${name}" namespace="$(arg namespace)" parent="${parent}" xyz="0.13 0 0.068" rpy="0 0 ${M_PI}"/>
+    <xacro:car_chassis name="${name}" parent="${parent}" xyz="0.13 0 0.068" rpy="0 0 ${M_PI}"/>
     <!-- Wheel -->
-    <xacro:wheel namespace="$(arg namespace)" side="rear_left"   parent="${parent}"   xyz="0    -0.055 ${wheel_radius}" rpy="+${pi/2} 0 0" radius="${wheel_radius}"  steering="fixed"/>
-    <xacro:wheel namespace="$(arg namespace)" side="rear_right"  parent="${parent}"   xyz="0    +0.055 ${wheel_radius}" rpy="-${pi/2} 0 0" radius="${wheel_radius}"  steering="fixed"/>
-    <xacro:wheel namespace="$(arg namespace)" side="front_left"  parent="${parent}"   xyz="0.26 -0.055 ${wheel_radius}" rpy="+${pi/2} 0 0" radius="${wheel_radius}"  steering="revolute"/>
-    <xacro:wheel namespace="$(arg namespace)" side="front_right" parent="${parent}"   xyz="0.26 +0.055 ${wheel_radius}" rpy="-${pi/2} 0 0" radius="${wheel_radius}"  steering="revolute"/>
+    <xacro:wheel side="rear_left"   parent="${parent}"   xyz="0    -0.055 ${wheel_radius}" rpy="+${pi/2} 0 0" radius="${wheel_radius}"  steering="fixed"/>
+    <xacro:wheel side="rear_right"  parent="${parent}"   xyz="0    +0.055 ${wheel_radius}" rpy="-${pi/2} 0 0" radius="${wheel_radius}"  steering="fixed"/>
+    <xacro:wheel side="front_left"  parent="${parent}"   xyz="0.26 -0.055 ${wheel_radius}" rpy="+${pi/2} 0 0" radius="${wheel_radius}"  steering="revolute"/>
+    <xacro:wheel side="front_right" parent="${parent}"   xyz="0.26 +0.055 ${wheel_radius}" rpy="-${pi/2} 0 0" radius="${wheel_radius}"  steering="revolute"/>
     <!-- Motor plugin -->
-    <xacro:wheels_steering namespace="$(arg namespace)" radius="${wheel_radius}"/>
-	<xacro:car_state_publisher namespace="$(arg namespace)"/>
+    <xacro:wheels_steering radius="${wheel_radius}"/>
+    <!-- <xacro:sensor_d435 name="$(arg name)" topics_ns="$(arg topics_ns)" parent="${parent}" use_nominal_extrinsics="$(arg use_nominal_extrinsics)"
+    publish_pointcloud="$(arg publish_pointcloud)" add_plug="$(arg add_plug)">
+      <origin xyz="0 0 0.18" rpy="0 0.1 0"/>
+    </xacro:sensor_d435>
+ -->
+  <xacro:sensor_d435 name="$(arg name)" topics_ns="$(arg topics_ns)" parent="chassis" use_nominal_extrinsics="$(arg use_nominal_extrinsics)" publish_pointcloud="$(arg publish_pointcloud)" add_plug="$(arg add_plug)">
+    <origin xyz="0.13 0 0.12" rpy="0 0.1 3.14159"/>
+  </xacro:sensor_d435>
   </xacro:macro>
 </robot>

File: car_gazebo_models/models/platforms/car/body/chassis.xacro (robot description, xacro)
@@ -1,5 +1,5 @@
 <?xml version="1.0"?>
 <robot xmlns:xacro="http://ros.org/wiki/xacro">
-  <xacro:macro name="car_chassis" params="name namespace parent xyz rpy">
+  <xacro:macro name="car_chassis" params="name parent xyz rpy">
   <xacro:property name="plate_x"    value="0.26" />
   <xacro:property name="plate_y"    value="0.08" />
@@ -8,8 +8,8 @@
     <joint name="${parent}_${name}_joint" type="fixed">
         <origin xyz="${xyz}" rpy="${rpy}"/>
-        <parent link="${namespace}/${parent}"/>
-        <child link="${namespace}/${name}"/>
+        <parent link="${parent}"/>
+        <child link="${name}"/>
     </joint>
-    <link name="${namespace}/${name}">
+    <link name="${name}">
         <visual>
             <origin xyz="${plate_x/2} 0 -${plate_z}" rpy="0 0 0"/>

File: car_gazebo_models/models/platforms/car/body/wheel.xacro (robot description, xacro)
@@ -1,5 +1,5 @@
 <?xml version="1.0"?>
 <robot xmlns:xacro="http://ros.org/wiki/xacro">
-  <xacro:macro name="wheel" params="side namespace parent xyz rpy radius steering">
+  <xacro:macro name="wheel" params="side parent xyz rpy radius steering">
     <xacro:property name="mount_size" value="0.01" />
     <xacro:property name="steering_length" value="0.03" />
@@ -14,10 +14,10 @@
     <joint name="wheel_mount_${side}_joint" type="${steering}">  <!--fixed/revolute -->
         <origin xyz="${xyz}" rpy="${rpy}"/>
-        <parent link="${namespace}/${parent}"/>
-        <child link="${namespace}/wheel_mount_${side}"/>
+        <parent link="${parent}"/>
+        <child link="wheel_mount_${side}"/>
         <axis xyz="0 1 0"/>
         <limit effort="50" velocity="50" lower= "${-M_PI}" upper="${M_PI}" />
     </joint>
-    <link name="${namespace}/wheel_mount_${side}">
+    <link name="wheel_mount_${side}">
         <visual>
             <origin xyz="0 0 ${mount_size/2}" rpy="0 0 0"/>
@@ -30,8 +30,8 @@
     <joint name="wheel_steering_${side}_joint" type="fixed">
         <origin xyz=" 0 0 0" rpy="0 0 0"/>
-        <parent link="${namespace}/wheel_mount_${side}"/>
-        <child link="${namespace}/wheel_steering_${side}"/>
+        <parent link="wheel_mount_${side}"/>
+        <child link="wheel_steering_${side}"/>
     </joint>
-    <link name="${namespace}/wheel_steering_${side}">
+    <link name="wheel_steering_${side}">
         <inertial>
             <mass value="0.001"/>
@@ -58,10 +58,10 @@
     <joint name="wheel_axis_${side}_joint" type="continuous">
         <origin xyz=" 0 0 ${steering_radius}" rpy="0 0 0"/>
-        <parent link="${namespace}/wheel_steering_${side}"/>
-        <child link="${namespace}/wheel_axis_${side}"/>
+        <parent link="wheel_steering_${side}"/>
+        <child link="wheel_axis_${side}"/>
         <axis xyz="0 0 1"/>
           <dynamics damping="0.000" friction="0.0"/>
     </joint>
-    <link name="${namespace}/wheel_axis_${side}">
+    <link name="wheel_axis_${side}">
         <visual>
             <origin xyz="0 0 ${axis_length/2}" rpy="0 0 0"/>
@@ -83,8 +83,8 @@
     <joint name="wheel_${side}_joint" type="fixed">
         <origin xyz=" 0 0 ${axis_length}" rpy="0 0 0"/>
-        <parent link="${namespace}/wheel_axis_${side}"/>
-        <child link="${namespace}/wheel_${side}"/>
+        <parent link="wheel_axis_${side}"/>
+        <child link="wheel_${side}"/>
     </joint>
-    <link name="${namespace}/wheel_${side}">
+    <link name="wheel_${side}">
         <visual>
             <origin xyz="0 0 ${wheel_length/2}" rpy="0 0 0"/>
@@ -106,8 +106,8 @@
     <joint name="wheel_cap_${side}_joint" type="fixed">
         <origin xyz=" 0 0 ${wheel_length}" rpy="0 0 0"/>
-        <parent link="${namespace}/wheel_${side}"/>
-        <child link="${namespace}/wheel_cap_${side}"/>
+        <parent link="wheel_${side}"/>
+        <child link="wheel_cap_${side}"/>
     </joint>
-    <link name="${namespace}/wheel_cap_${side}">
+    <link name="wheel_cap_${side}">
         <visual>
             <origin xyz="0 0 ${cap_length/2}" rpy="0 0 0"/>

File: car_gazebo_models/models/platforms/car/main.xacro (robot description, xacro)
@@ -10,4 +10,17 @@
   <xacro:property name="model_dir" value="$(arg model_dir)/$(arg platform_dir)/body"/>
   <xacro:include filename="${model_dir}/body.xacro"/>
-  <xacro:car_body name="chassis" namespace="$(arg namespace)" parent="base_link"/>
+  <xacro:car_body name="chassis" parent="base_link"/>
+  <!-- <xacro:include filename="$(find realsense2_description)/urdf/test_d435_camera.urdf.xacro" />
+	<sensor_d435 parent="chassis" xyz="0 -0.055 1">
+	</sensor_d435> -->
+  <!-- <xacro:include filename="$(find realsense2_description)/urdf/test_d435_camera.urdf.xacro" >
+    <pose>0.2 0 0.2 0 0 0</pose>
+  </xacro:include>
+  <joint name="camera_chassis_joint" type="fixed">
+    <child>realsense2_camera::link</child>
+    <parent>chassis</parent>
+    <parent link="chassis"/>
+    <child link="camera"/>
+  </joint> -->
+	<xacro:car_state_publisher robot_namespace="$(arg namespace)"/>
 </robot>

File: car_gazebo_models/models/platforms/car/plugins.xacro (robot description, xacro)
@@ -1,26 +1,27 @@
 <?xml version="1.0"?>
 <robot xmlns:xacro="http://ros.org/wiki/xacro">
-  <xacro:macro name="car_state_publisher" params="namespace">
-    <xacro:property name="robot_namespace" value="${namespace}" />
-    <gazebo>
-      <plugin name="joint_state_publisher" filename="libgazebo_ros_joint_state_publisher.so">
-        <robotNamespace>${robot_namespace}</robotNamespace>
-        <jointName> wheel_axis_rear_left_joint, wheel_axis_rear_right_joint, wheel_axis_front_left_joint, wheel_axis_front_right_joint, wheel_mount_front_left_joint, wheel_mount_front_right_joint</jointName>
-        <updateRate>25.0</updateRate>
-        <alwaysOn>true</alwaysOn>
-      </plugin>
-    </gazebo>
+  <xacro:macro name="car_state_publisher" params="robot_namespace">
+  	<gazebo>
+  		<plugin name="joint_state_publisher" filename="libgazebo_ros_joint_state_publisher.so">
+  			<robotNamespace>${robot_namespace}</robotNamespace>
+  			<jointName> wheel_axis_rear_left_joint, wheel_axis_rear_right_joint, wheel_axis_front_left_joint,
+        wheel_axis_front_right_joint, wheel_mount_front_left_joint, wheel_mount_front_right_joint
+        </jointName>
+  			<updateRate>1000.0</updateRate>
+  			<alwaysOn>true</alwaysOn>
+  		</plugin>
+  	</gazebo>
   </xacro:macro>
-  <xacro:macro name="wheels_steering" params="namespace radius">
-    <xacro:property name="wheel_radius" value="${radius}" />
+  <xacro:macro name="wheels_steering" params="radius">
+  <xacro:property name="wheel_radius" value="${radius}" />
     <gazebo>
         <plugin name="wheels_steering_controller" filename="libgazebo_ros_wheels_steerable.so">
             <rosDebugLevel>Debug</rosDebugLevel>
+            <rosDebugLevel>Debug</rosDebugLevel>
             <topicOdom>odom</topicOdom>
             <frameOdom>odom</frameOdom>
-            <publishOdomTF>true</publishOdomTF>
             <topicGroundTruth>ground_truth</topicGroundTruth>
             <frameGroundTruth>ground_truth</frameGroundTruth>
-            <frameBase>base_link</frameBase>
+            <frameBase>odom</frameBase>
             <topicTwist>cmd_vel</topicTwist>
             <jointRearLeft>wheel_axis_rear_left_joint</jointRearLeft>
@@ -35,5 +36,4 @@
             <maxSteeringAngle>0.5235987756</maxSteeringAngle>
             <!--PID controller parameter-->
-            <updateRateController>100</updateRateController>
             <maxEffortSteeringPid>5.12</maxEffortSteeringPid>
             <pidP>15.0</pidP>
